Commit message: bug fix

File: src/chassis/andino_description/urdf/include/andino_control.urdf.xacro (robot description, xacro)
@@ -17,4 +17,6 @@
         <param name="enc_ticks_per_rev">${hardware_props['enc_ticks_per_rev']}</param>
         <param name="can_channel">${hardware_props['can_channel']}</param>
+        <param name="left_motor_id">${hardware_props['left_motor_id']}</param>
+        <param name="right_motor_id">${hardware_props['right_motor_id']}</param>
       </hardware>
       <joint name="left_wheel_joint">

File: src/chassis/andino_description/urdf/include/common_sensors.urdf.xacro (robot description, xacro)
@@ -80,5 +80,5 @@
     <parent link="${parent_link}"/>
     <child link="camera_link"/>
-    <origin xyz="${sensor_prop['camera']['dx']} ${sensor_prop['camera']['dy']} ${sensor_prop['camera']['dz']}" rpy="0 0 0"/>
+    <origin xyz="${sensor_prop['camera']['dx']} ${sensor_prop['camera']['dy']} ${sensor_prop['camera']['dz']}" rpy="${sensor_prop['camera']['roll']} ${sensor_prop['camera']['pitch']} ${sensor_prop['camera']['yaw']}"/>
     <axis xyz="0 1 0" />
   </joint>
